Commit message: refact/moveit

File: manipulate/moveit_config/config/left_walkie_arm.ros2_control.xacro (robot description, xacro)
@@ -71,9 +71,9 @@
                 <state_interface name="effort"/>
             </joint>
-            <joint name="left_gripper_worm_gear">
+            <joint name="left_gripper_worm_gear_joint">
                 <command_interface name="position"/>
                 <command_interface name="effort"/>
                 <state_interface name="position">
-                  <param name="initial_value">${initial_positions['left_gripper_worm_gear']}</param>
+                  <param name="initial_value">${initial_positions['left_gripper_worm_gear_joint']}</param>
                 </state_interface>
                 <state_interface name="velocity"/>
